File: pcbs/PlusCart/PlusCart.sch (EAGLE design)
At the start: 5 parts, among them CON3 A2600

Commit message: Breakoutboard optimization, new gerberfiles
Parts:
- added JP5: (no value), pinhead:PINHD-2X8
- added JP6: (no value), pinhead:PINHD-2X4
- JP1: device pinhead:PINHD-2X16 -> pinhead:PINHD-2X2
- JP2: device pinhead:PINHD-2X12 -> pinhead:PINHD-2X4
- JP3: device pinhead:PINHD-2X18 -> pinhead:PINHD-2X3
- JP4: device pinhead:PINHD-2X4 -> pinhead:PINHD-2X9
Connections:
- removed net N$1: JP3.35, JP3.36
- net +3V3: now also JP1.2, JP4.4, JP5.2, JP6.2, JP6.6; no longer JP1.30, JP2.10, JP3.8, JP4.2, JP4.6
- net A0: now also JP2.2; no longer JP1.16
- net A1: now also JP2.1; no longer JP1.15
- net A10: now also JP4.9; no longer JP2.15
- net A11: now also JP4.12; no longer JP2.18
- net A12: now also JP4.11; no longer JP2.17
- net A2: now also JP2.4; no longer JP1.18
- net A3: now also JP2.3; no longer JP1.17
- net A4: now also JP2.6; no longer JP1.20
- net A5: now also JP2.5; no longer JP1.19
- net A6: now also JP2.8; no longer JP1.22
- net A7: now also JP2.7; no longer JP1.21
- net A8: now also JP4.7; no longer JP2.13
- net A9: now also JP4.10; no longer JP2.16
- net D0: now also JP5.4; no longer JP3.10
- net D1: now also JP5.3; no longer JP3.9
- net D2: now also JP5.6; no longer JP3.12
- net D3: now also JP5.10; no longer JP3.16
- net D4: now also JP5.16; no longer JP3.22
- net D5: now also JP5.15; no longer JP3.21
- net D6: now also JP4.15; no longer JP2.21
- net D7: now also JP4.18; no longer JP2.24
- net GND: now also JP1.3, JP3.1, JP4.13, JP4.14, JP4.16, JP4.2, JP5.1, JP6.7; no longer JP1.29, JP1.31, JP2.19, JP2.20, JP2.22, JP2.8, JP3.7, JP4.7
- net USART1_RX: now also JP3.5, JP6.8; no longer JP1.5, JP4.8
- net USART1_TX: now also JP3.6, JP6.1; no longer JP1.6, JP4.1
- net VCC: now also JP1.4; no longer JP1.2, JP1.32
